File: kicad/IN12B Breakout horizontal.kicad_pcb (KiCad board)
At the start: 2 copper layers, 31.5 x 36.8 mm, 3 parts, among them J1 Conn_01x12_Male

Commit message: finished rev.A PCBs
Parts:
- moved G*** 20.9 mm to (88.7, 69.2)
Routing:
- net /C6: track 0.00 -> 43.0 mm, vias 0 -> 1
- net /C5: track 0.00 -> 35.5 mm, vias 0 -> 1
- net /C7: track 0.00 -> 33.1 mm, vias 0 -> 1
- net /C4: track 0.00 -> 31.7 mm, vias 0 -> 1
- net /C8: track 0.00 -> 28.2 mm, vias 0 -> 1
- net /C3: track 0.00 -> 27.8 mm, vias 0 -> 1
- net /C9: track 0.00 -> 25.0 mm, vias 0 -> 1
- net /C2: track 0.00 -> 24.2 mm, vias 0 -> 1
- net /CDot: track 0.00 -> 21.8 mm, vias 0 -> 1
- net /C0: track 0.00 -> 21.5 mm, vias 0 -> 1
- net /A: track 0.00 -> 20.1 mm, vias 0 -> 1
- net /C1: track 0.00 -> 19.0 mm, vias 0 -> 1
