File: kicad/IN12B Breakout vertical.kicad_pcb (KiCad board)
At the start: 2 copper layers, 29.2 x 33 mm, 3 parts, among them J1 Conn_01x12_Male

Commit message: introduced horizontal and vertical PCB versions
Parts:
- moved G*** 0.43 mm to (107.5, 47.5), turned to 180 degrees
Other:
- board text added: "rev.A 07 21"
- board text added: "⊙"
- board text removed: "rev.A 07/21"
